File: SignalMast-Searchlight-SingleHead.brd (EAGLE design)
At the start: 12.7 x 50 mm, 2 parts

Commit message: normalized values
Parts:
- CON1: value (none) -> 2x3-0.100
- LED1: value LED-APA102 -> RGB
Changed lines of the file:
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@@
 </autorouter>
 <elements>
-<element name="CON1" library="SPCoast" package="2X3-SMD_EDGE" value="" x="6.35" y="1.905"/>
-<element name="LED1" library="SPCoast" package="APA102" value="LED-APA102" x="4.445" y="42.926" smashed="yes">
+<element name="CON1" library="SPCoast" package="2X3-SMD_EDGE" value="2x3-0.100" x="6.35" y="1.905"/>
+<element name="LED1" library="SPCoast" package="APA102" value="RGB" x="4.445" y="42.926" smashed="yes">
 <attribute name="HEIGHT" value="1mm" x="4.445" y="42.926" size="1.778" layer="27" font="vector" ratio="10" display="off"/>
 <attribute name="MOUSER_PRICE-STOCK" value="https://www.mouser.com/Search/Refine.aspx?Keyword=474-COM-14608" x="4.445" y="42.926" size="1.778" layer="27" font="vector" ratio="10" display="off"/>
