File: SignalMast-Searchlight-SingleHead.sch (EAGLE design)
At the start: 2 parts

Commit message: normalized values
Parts:
- CON1: value (none) -> 2x3-0.100
- LED1: value LED-APA102 -> RGB
Changed lines of the file:
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@@
 <parts>
 <part name="FRAME1" library="SPCoast" deviceset="DOC-FRAME-LETTER" device=""/>
-<part name="CON1" library="SPCoast" deviceset="CONNECTOR-M06" device="2X3-SMD"/>
-<part name="LED1" library="SPCoast" deviceset="LED-APA102" device=""/>
+<part name="CON1" library="SPCoast" deviceset="CONNECTOR-M06" device="2X3-SMD" value="2x3-0.100"/>
+<part name="LED1" library="SPCoast" deviceset="LED-APA102" device="" value="RGB"/>
 </parts>
 <sheets>
